Commit message: 整理旧版本xbot1的单板驱动程序

File: xbot_description/urdf/robot.xacro (robot description, xacro)
@@ -7,6 +7,6 @@
   <xacro:include filename="$(find xbot_description)/urdf/sick_tim.urdf.xacro" />
   <!-- Choose your laser -->
-  <xacro:sick_tim571 name="laser" ros_topic="scan"   />
-  <!-- <xacro:rplidarA2 name="laser" ros_topic="scan"   /> -->
+  <!--<xacro:sick_tim571 name="laser" ros_topic="scan"   />-->
+  <xacro:rplidarA2 name="laser" ros_topic="scan"   />
   <xacro:include filename="$(find xbot_description)/urdf/materials.xacro" />
   <xacro:include filename="$(find xbot_description)/urdf/xbot-u.urdf.xacro" />

File: xbot_description/urdf/sick_tim.urdf.xacro (robot description, xacro)
@@ -6,6 +6,6 @@
   <xacro:macro name="rplidarA2" params="name ros_topic">
     <xacro:sick_tim name="${name}" ros_topic="${ros_topic}"
-      length="0.06" width="0.06" height="0.079" mass="0.150" z_offset="0.0308"
-      min_range="0.2" max_range="12.0"
+      length="0.06" width="0.06" height="0.079" mass="0.150" z_offset="0.05595"
+      min_range="0.2" max_range="8.0"
       mesh="package://xbot_description/models/meshes/rplidar.dae" />
   </xacro:macro>
@@ -24,5 +24,5 @@
   <xacro:macro name="sick_tim571" params="name ros_topic">
     <xacro:sick_tim name="${name}" ros_topic="${ros_topic}"
-      length="0.06" width="0.06" height="0.086" mass="0.250" z_offset="0.05"
+      length="0.06" width="0.06" height="0.086" mass="0.250" z_offset="0.02"
       min_range="0.05" max_range="25.0"
       mesh="package://xbot_description/models/meshes/sick_tim571.stl" />
@@ -33,5 +33,5 @@
       <parent link="${name}_mount_link" />
       <child link="${name}" />
-      <origin rpy="0 0 3.1415926" xyz="0 0 ${z_offset}"/>
+      <origin rpy="0 0 0" xyz="0 0 ${z_offset}"/>
     </joint>
     <link name="${name}">

File: xbot_description/urdf/xbot-u.urdf.xacro (robot description, xacro)
@@ -66,5 +66,5 @@
     <parent link="base_link"/>
     <child link="laser_mount_link"/>
-    <origin rpy="0 0 0" xyz=".120 0 .205"/>
+    <origin rpy="0 0 0" xyz=".114 0 .17"/>
   </joint>
   <link name="imu_link"/>
@@ -73,5 +73,5 @@
     <parent link="base_link"/>
     <child link="imu_link"/>
-    <origin rpy="0 0 0" xyz="0.0454 -0.0157 1.1724"/>
+    <origin rpy="0 0 0" xyz="0 0 .2"/>
   </joint>
   <link name="left_wheel">
@@ -152,5 +152,5 @@
     <parent link="base_link"/>
     <child link="yaw_platform"/>
-    <origin rpy="0 0 0" xyz="0 0 1.232"/>
+    <origin rpy="0 0 0" xyz="0 0 1.305"/>
     <limit effort="100" velocity="100" lower="-1.57" upper="1.57" />
     <dynamics damping="0.0" friction="10.0"/>
@@ -179,5 +179,5 @@
     <parent link="yaw_platform"/>
     <child link="pitch_platform"/>
-    <origin rpy="0 0 0" xyz="0.0208 0 0.01325"/>
+    <origin rpy="0 0 0" xyz="0 0 0"/>
     <limit effort="100" velocity="100" lower="-1.57" upper="1.57" />
     <dynamics damping="0.0" friction="10.0"/>

Commit message: release 3.2.4

File: xbot_description/urdf/robot.xacro (robot description, xacro)
@@ -4,8 +4,10 @@
   xmlns:sensor="http://playerstage.sourceforge.net/gazebo/xmlschema/#sensor"
   xmlns:xacro="http://ros.org/wiki/xacro"
-  name="sick_tim">
-  <xacro:include filename="$(find xbot_description)/urdf/sick_tim.urdf.xacro" />
+  name="xbot">
+  <xacro:include filename="$(find xbot_description)/urdf/_d415.urdf.xacro" />
+  <xacro:include filename="$(find xbot_description)/urdf/laser.urdf.xacro" />
   <!-- Choose your laser -->
-  <xacro:sick_tim571 name="laser" ros_topic="scan"   />
+  <xacro:rplidarA2 name="laser" ros_topic="scan">
+  </xacro:rplidarA2>
   <!-- <xacro:rplidarA2 name="laser" ros_topic="scan"   /> -->
   <xacro:include filename="$(find xbot_description)/urdf/materials.xacro" />
@@ -13,3 +15,6 @@
   <xacro:include filename="$(find xbot_description)/urdf/xbot-u.gazebo" />
   <xacro:xbot_base/>
+  <xacro:sensor_d415 parent="camera_mount_link">
+    <origin xyz="0 0 0" rpy="0 0 0"/>
+  </xacro:sensor_d415>
 </robot>

File: xbot_description/urdf/xbot-u.urdf.xacro (robot description, xacro)
@@ -19,8 +19,13 @@
     </inertial>
     <visual>
-      <origin xyz="0 0 0" rpy="0 0 0" />
-      <geometry>
-        <mesh filename="package://xbot_description/models/meshes/base_link.dae" />
-      </geometry>
+      <origin xyz="0 0 0.01" rpy="1.5707 0 -1.5707" />
+      <geometry>
+        <mesh filename="package://xbot_description/models/xbot/bace.dae" />
+      </geometry>
+      <material
+        name="">
+        <color
+          rgba="0.2 0.2 0.2 1.0" />
+      </material>
     </visual>
     <collision name="front_omniwheel">
@@ -66,5 +71,5 @@
     <parent link="base_link"/>
     <child link="laser_mount_link"/>
-    <origin rpy="0 0 0" xyz=".120 0 .205"/>
+    <origin rpy="0 0 0" xyz="0.120 0 0.2"/>
   </joint>
   <link name="imu_link"/>
@@ -73,5 +78,5 @@
     <parent link="base_link"/>
     <child link="imu_link"/>
-    <origin rpy="0 0 0" xyz="0.0454 -0.0157 1.1724"/>
+    <origin rpy="0 0 0" xyz="0.04548 -0.01552 1.1695"/>
   </joint>
   <link name="front_echo_link"/>
@@ -80,5 +85,5 @@
     <parent link="base_link"/>
     <child link="front_echo_link"/>
-    <origin rpy="0 0 0" xyz="0.236 0.0 0.05683"/>
+    <origin rpy="0 0 0" xyz="0.236 0.0 0.087"/>
   </joint>
   <link name="rear_echo_link"/>
@@ -87,5 +92,5 @@
     <parent link="base_link"/>
     <child link="rear_echo_link"/>
-    <origin rpy="0 0 1.5707" xyz="-0.236 0.0 0.05683"/>
+    <origin rpy="0 0 1.5707" xyz="-0.236 0.0 0.087"/>
   </joint>
   <link name="left_wheel">
@@ -99,5 +104,5 @@
       <origin xyz="0 0 0" rpy="0 0 -1.57079632"/>
       <geometry>
-        <mesh filename="package://xbot_description/models/meshes/wheel.dae" />
+        <mesh filename="package://xbot_description/models/xbot/wheel.dae" />
       </geometry>
     </visual>
@@ -110,5 +115,5 @@
   <joint type="continuous" name="left_wheel_hinge">
     <axis xyz="0 1 0" rpy="0 0 0"/>
-    <origin xyz="0 0.23 .095" rpy="0 0 0"/>
+    <origin xyz="0 0.2289 0.095" rpy="0 0 0"/>
     <parent link="base_link"/>
     <child link="left_wheel"/>
@@ -126,5 +131,5 @@
       <origin xyz="0 0 0" rpy="0 0 1.57079632"/>
       <geometry>
-        <mesh filename="package://xbot_description/models/meshes/wheel.dae" />
+        <mesh filename="package://xbot_description/models/xbot/wheel.dae" />
       </geometry>
     </visual>
@@ -137,5 +142,5 @@
   <joint type="continuous" name="right_wheel_hinge">
     <axis xyz="0 1 0" rpy="0 0 0"/>
-    <origin xyz="0 -0.23 .095" rpy="0 0 0"/>
+    <origin xyz="0 -0.2289 0.095" rpy="0 0 0"/>
     <parent link="base_link"/>
     <child link="right_wheel"/>
@@ -150,8 +155,16 @@
     </inertial>
     <visual>
-      <origin xyz="0 0 0" rpy="0 0 1.57079632" />
-      <geometry>
-        <mesh filename="package://xbot_description/models/meshes/yaw_platform.dae" />
-      </geometry>
+      <origin
+        xyz="0 0 0"
+        rpy="0 0 0" />
+      <geometry>
+        <mesh
+          filename="package://xbot_description/models/xbot/head_yaw_link.STL" />
+      </geometry>
+      <material
+        name="">
+        <color
+          rgba="0.2 0.2 0.2 1.0" />
+      </material>
     </visual>
     <collision>
@@ -166,5 +179,5 @@
     <parent link="base_link"/>
     <child link="yaw_platform"/>
-    <origin rpy="0 0 0" xyz="0 0 1.232"/>
+    <origin xyz="0 0 1.222" rpy="0 0 0"/>
     <limit effort="100" velocity="100" lower="-1.57" upper="1.57" />
     <dynamics damping="0.0" friction="10.0"/>
@@ -177,8 +190,16 @@
     </inertial>
     <visual>
-      <origin xyz="0 0 0" rpy="0 0 0" />
-      <geometry>
-        <mesh filename="package://xbot_description/models/meshes/pitch_platform.dae" />
-      </geometry>
+      <origin
+        xyz="0 0 0"
+        rpy="0 1.5707 0" />
+      <geometry>
+        <mesh
+          filename="package://xbot_description/models/xbot/pitch.dae" />
+      </geometry>
+      <material
+        name="">
+        <color
+          rgba="0.3 0.3 0.3 1.0" />
+      </material>
     </visual>
     <collision>
@@ -190,37 +211,18 @@
   </link>
   <joint name="yaw_to_pitch_platform" type="revolute">
-    <axis xyz="0 1 0"/>
+    <axis xyz="0 0 1"/>
     <parent link="yaw_platform"/>
     <child link="pitch_platform"/>
-    <origin rpy="0 0 0" xyz="0.0208 0 0.01325"/>
-    <limit effort="100" velocity="100" lower="-1.57" upper="1.57" />
+    <origin rpy="1.5708 0 0" xyz="0.0208 0.0013 0.01425"/>
+    <limit effort="100" velocity="100" lower="-1.047" upper="0.52" />
     <dynamics damping="0.0" friction="10.0"/>
   </joint>
   <!-- Camera -->
-  <link name="camera_link">
-    <collision>
-      <origin xyz="0 0 0" rpy="0 0 0"/>
-      <geometry>
-        <box size="0.1 0.1 0.1"/>
-      </geometry>
-    </collision>
-    <visual>
-      <origin xyz="0 0 0" rpy="0 0 0"/>
-      <geometry>
-        <!--<mesh filename="package://xbot_description/models/meshes/xtion_pro_camera.dae" />-->
-        <mesh filename="package://xbot_description/models/meshes/realsense.dae" />
-      </geometry>
-    </visual>
-    <inertial>
-      <mass value="1e-5" />
-      <origin xyz="0 0 0" rpy="0 0 0"/>
-      <inertia ixx="1e-6" ixy="0" ixz="0" iyy="1e-6" iyz="0" izz="1e-6" />
-    </inertial>
-  </link>
-  <joint name="camera_joint" type="fixed">
-    <axis xyz="0 1 0" />
-    <origin xyz="-0.005 0 .06" rpy="0 0 0"/>
+  <link name="camera_mount_link" />
+  <joint name="pitch2camera_joint" type="fixed">
+    <axis xyz="0 0 0" />
+    <origin xyz="-0.005 0.035 0.0" rpy="-1.5708 0 0"/>
     <parent link="pitch_platform"/>
-    <child link="camera_link"/>
+    <child link="camera_mount_link"/>
   </joint>
   </xacro:macro>
